File: mpg_pinout/mpg_pinout.kicad_pcb (KiCad board)
At the start: 2 copper layers, 9 parts, among them J1 Conn_02x05_Odd_Even, J2 Conn_01x02_Pin, J3 Conn_01x02_Pin, J4 Conn_01x02_Pin, J5 Conn_01x02_Pin, J6 Conn_01x02_Pin, J7 Conn_01x02_Pin, J8 Conn_01x02_Pin

Commit message: third commit
Parts:
- added R2: R, Resistor_THT:R_Axial_DIN0414_L11.9mm_D4.5mm_P15.24mm_Horizontal, F.Cu at (78.7, 61.0)
- added R3: R, Resistor_THT:R_Axial_DIN0414_L11.9mm_D4.5mm_P15.24mm_Horizontal, F.Cu at (78.7, 66.0)
- added R4: R, Resistor_THT:R_Axial_DIN0414_L11.9mm_D4.5mm_P25.40mm_Horizontal, F.Cu at (104.1, 76.2)
- added R5: R, Resistor_THT:R_Axial_DIN0414_L11.9mm_D4.5mm_P15.24mm_Horizontal, F.Cu at (104.1, 71.1)
- added R6: R, Resistor_THT:R_Axial_DIN0414_L11.9mm_D4.5mm_P15.24mm_Horizontal, F.Cu at (106.9, 83.8)
- moved J1 18.8 mm to (84.1, 91.4)
- moved R1 5.64 mm to (104.1, 45.7)
- moved J8 3.31 mm to (111.8, 106.7)
- moved J7 2.81 mm to (111.8, 96.5)
- moved J6 2.30 mm to (111.8, 86.4)
- moved J5 1.80 mm to (111.8, 76.2)
- moved J4 1.30 mm to (111.8, 66.0)
- moved J2 0.80 mm to (111.8, 55.9)
- moved J3 0.36 mm to (111.8, 45.7)
Connections:
- J4 pad 1: Net-(J1-Pin_5) -> Net-(J4-Pin_1)
- J4 pad 2: Net-(J1-Pin_6) -> Net-(J4-Pin_2)
- J5 pad 1: Net-(J1-Pin_4) -> Net-(J5-Pin_1)
- J5 pad 2: Net-(J1-Pin_3) -> Net-(J5-Pin_2)
- J6 pad 2: Net-(J1-Pin_7) -> Net-(J6-Pin_2)
Routing:
- net Net-(J1-Pin_8): track 0.00 -> 43.5 mm
- net Net-(J1-Pin_7): track 0.00 -> 43.4 mm
- net Net-(J6-Pin_2): track 0.00 -> 43.2 mm
- net Net-(J1-Pin_6): track 0.00 -> 38.7 mm
- net Net-(J1-Pin_3): track 0.00 -> 38.4 mm
- net Net-(J5-Pin_2): track 0.00 -> 38.1 mm
- net Net-(J1-Pin_9): track 0.00 -> 31.3 mm
- net Net-(J1-Pin_10): track 0.00 -> 27.3 mm
- net Net-(J1-Pin_5): track 0.00 -> 25.7 mm
- net Net-(J1-Pin_1): track 38.7 -> 63.2 mm
- net unconnected-(J1-Pin_2-Pad2): track 111.0 -> 135.1 mm
- net Net-(J4-Pin_1): track 0.00 -> 22.9 mm
- net Net-(J5-Pin_1): track 0.00 -> 18.5 mm
- net Net-(J1-Pin_4): track 0.00 -> 14.8 mm
- net Net-(J4-Pin_2): track 0.00 -> 7.62 mm
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
Commit message: Made pdf file for mpg and bidirectional, 7x10cm
Parts:
- added H1: MountingHole, _customized:hole_3mm, F.Cu at (30.5, 30.5)
- added H2: MountingHole, _customized:hole_3mm, F.Cu at (30.5, 91.4)
- added H3: MountingHole, _customized:hole_3mm, F.Cu at (92.5, 43.2)
- added H4: MountingHole, _customized:hole_3mm, F.Cu at (105.2, 43.4)
- added H5: MountingHole, _customized:hole_3mm, F.Cu at (105.4, 78.7)
- added H6: MountingHole, _customized:hole_3mm, F.Cu at (92.5, 78.7)
- added J10: Conn_01x10, _customized:connector_01x10_508, F.Cu at (118.1, 38.1)
- added J9: Conn_01x10, _customized:connector_01x10_508, F.Cu at (80.0, 38.1)
- added R7: R, Resistor_THT:R_Axial_DIN0411_L9.9mm_D3.6mm_P25.40mm_Horizontal, F.Cu at (98.4, 48.5)
- added U1: ~, _customized:TXS0108, F.Cu at (92.5, 49.5)
- moved J1 49.1 mm to (38.4, 73.7)
- moved J2 49.1 mm to (66.0, 38.1)
- moved J3 49.1 mm to (66.0, 27.9)
- moved J4 49.1 mm to (66.0, 48.3)
- moved J5 49.1 mm to (66.0, 58.4)
- moved J6 49.1 mm to (66.0, 68.6)
- moved J7 49.1 mm to (66.0, 78.7)
- moved J8 49.1 mm to (66.0, 88.9)
- moved R1 49.1 mm to (58.4, 27.9)
- moved R4 49.1 mm to (58.4, 58.4)
- moved R5 49.1 mm to (58.4, 53.3)
- moved R2 49.1 mm to (33.0, 43.2)
- moved R3 49.1 mm to (33.0, 48.3)
- moved R6 49.1 mm to (61.2, 66.0)
Routing:
- net Net-(J9-Pin_1): track 0.00 -> 29.5 mm
- net Net-(J10-Pin_1): track 0.00 -> 23.8 mm
- net Net-(J9-Pin_10): track 0.00 -> 23.8 mm
- net Net-(J10-Pin_2): track 0.00 -> 21.4 mm
- net Net-(J9-Pin_2): track 0.00 -> 21.0 mm
- net Net-(J10-Pin_3): track 0.00 -> 18.9 mm
- net Net-(J9-Pin_3): track 0.00 -> 18.8 mm
- net Net-(J10-Pin_10): track 0.00 -> 17.7 mm
- net Net-(J10-Pin_9): track 0.00 -> 16.6 mm
- net Net-(J9-Pin_9): track 0.00 -> 16.1 mm
- net Net-(J10-Pin_8): track 0.00 -> 15.6 mm
- net Net-(J9-Pin_8): track 0.00 -> 15.1 mm
- net Net-(J10-Pin_7): track 0.00 -> 14.5 mm
- net Net-(J10-Pin_4): track 0.00 -> 14.5 mm
- net Net-(J9-Pin_7): track 0.00 -> 14.0 mm
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